Commit message: fix wheelchair left and right swap in differential controller :bug:

File: simulation_ws/src/wheelchair/urdf/base.urdf.xacro (robot description, xacro)
@@ -62,7 +62,5 @@
       <xacro:caster_wheel_inertia />
       <visual>
-        <!-- <origin xyz="0 0 0" rpy="${PI/2} 0 0" /> -->
         <geometry>
-          <!-- <cylinder length="0.038" radius="${caster_wheel_radius}" /> -->
           <mesh filename="package://wheelchair/meshes/caster_wheel.dae" />
         </geometry>
@@ -72,5 +70,4 @@
         <geometry>
           <cylinder length="0.038" radius="${caster_wheel_radius}" />
-          <!-- <mesh filename="package://wheelchair/meshes/caster_wheel.dae" /> -->
          </geometry>
       </collision>
@@ -82,5 +79,4 @@
     <joint name="${parent}_${suffix}_caster_hub_joint" type="continuous" >
       <axis xyz="0 0 1" />
-      <!-- <limit lower="${PI}" upper="${-1*PI}" effort="0.0" velocity="0.0" /> -->
       <dynamics damping="0.0" friction="0.0" />
       <xacro:insert_block name="origin" />
@@ -103,5 +99,4 @@
     </link>
     <xacro:caster_hub_gazebo suffix="${suffix}" />
-    <!-- <xacro:caster_hub_transmission parent="${parent}" suffix="${suffix}" /> -->
   </xacro:macro>
   <!-- Macro for caster set (caster wheel & hub) -->

File: simulation_ws/src/wheelchair/urdf/wheelchair.gazebo.xacro (robot description, xacro)
@@ -36,6 +36,6 @@
         <alwaysOn>true</alwaysOn>
         <updateRate>50</updateRate>
-        <leftJoint>base_right_front_wheel_joint</leftJoint>
-        <rightJoint>base_left_front_wheel_joint</rightJoint>
+        <leftJoint>base_left_front_wheel_joint</leftJoint>
+        <rightJoint>base_right_front_wheel_joint</rightJoint>
         <wheelSeparation>${separation}</wheelSeparation>
         <wheelDiameter>${diameter}</wheelDiameter>
