Commit message: iss + woa + pso + add 3 worlds in simulation :fire:

File: simulation_ws/src/wheelchair/urdf/wheelchair.gazebo.xacro (robot description, xacro)
@@ -7,5 +7,6 @@
     <plugin name="gazebo_ros_control" filename="libgazebo_ros_control.so" />
       <plugin filename="libgazebo_ros_joint_state_publisher.so" name="joint_state_publisher">
-        <jointName>base_left_caster_hub_joint, base_right_caster_hub_joint, base_left_front_wheel_joint, base_right_front_wheel_joint, left_caster_hub_left_caster_wheel_joint, right_caster_hub_right_caster_wheel_joint</jointName>
+        <jointName>base_left_caster_hub_joint, base_right_caster_hub_joint, base_left_front_wheel_joint,
+        base_right_front_wheel_joint, left_caster_hub_left_caster_wheel_joint, right_caster_hub_right_caster_wheel_joint</jointName>
         <updateRate>50.0</updateRate>
         <alwaysOn>true</alwaysOn>
@@ -21,6 +22,6 @@
   <xacro:macro name="caster_wheel_gazebo" params="suffix" >
     <gazebo reference="${suffix}_caster_wheel_link" >
-      <mu1 value="100.0" />
-      <mu2 value="100.0" />
+      <mu1 value="1000.0" />
+      <mu2 value="1000.0" />
       <kd value="1.0" />
     </gazebo>

File: simulation_ws/src/wheelchair/urdf/wheelchair.hokuyo.xacro (robot description, xacro)
@@ -16,5 +16,5 @@
      <origin xyz="0 0 0" rpy="0 0 0"/>
      <geometry>
-        <box size="0.1 0.1 0.1"/>
+        <box size="0.1 0.1 0.05"/>
      </geometry>
    </collision>
@@ -41,10 +41,10 @@
           <samples>720</samples>
           <resolution>1</resolution>
-          <min_angle>1.570796</min_angle>
-          <max_angle>-1.570796</max_angle>
+          <min_angle>-1.570796</min_angle>
+          <max_angle>1.570796</max_angle>
         </horizontal>
       </scan>
       <range>
-        <min>0.08</min>
+        <min>0.1</min>
         <max>10.0</max>
         <resolution>0.01</resolution>
